File: pcb/rabbit-body/rabbit-body.kicad_pcb (KiCad board)
At the start: 4 copper layers, 120.5 x 269.9 mm, 116 parts, among them J1 XT60 BAT, J10 ToF, J11 ToF, J12 lidar C1, J13 bumpers front, J14 bumpers rear, J15 button, J16 status LED, J17 Jetson UART, J18 Pi fan 5V, J19 USB hub 7-36V, J2 RoboClaw B+/B-, J20 spare out, J21 XT30 JETSON, J22 servo 0, J23 servo 1, J24 servo 2, J25 servo 3, J3 Pi 40-pin, J4 RoboClaw I/O, J5 E-stop loop, J6 ENC left, J7 ENC right, J8 ToF, J9 ToF, Q1 AO3400A, Q2 AO3400A, Q3 AO3400A, U1 RoboClaw 2x30A, U2 Pololu 2813, U3 INA4235, U4 D24V90F5, U5 D36V50F12, U6 D36V50F6, U7 TPS73733, U8 PCA9685PW, U9 DS3231SN

Commit message: feat(hw): mounts for the 3-deck stack, PCB review fixes (TVS, ToF 3V3, motor star, ZED cutout)
Co-Authored-By: Claude Opus 5.5 <noreply@anthropic.com>
Claude-Session: https://claude.ai/code/session_01BqVLDBXG9mdqYKRp3kWsAJ
Parts:
- added D7: SMBJ20CA, Diode_SMD:D_SMB, F.Cu at (192.1, 232.2)
- NT1: footprint NetTie:NetTie-2_SMD_Pad2.0mm -> rabbit_body:NetTie_3.5mm
- moved Q3 3.00 mm to (180.0, 62.5)
- moved R24 3.00 mm to (176.0, 62.5)
- moved R25 3.00 mm to (180.0, 66.0)
- moved NT1 0.90 mm to (191.5, 256.5)
Routing:
- net +5V: track 251.0 -> 317.8 mm, vias 1 -> 0
- net GPIO12: track 64.2 -> 98.9 mm
- net GPIO16: track 100.4 -> 78.6 mm, vias 2 -> 1
- net BUMPER_REAR: track 207.4 -> 186.1 mm, vias 1 -> 0
- net BUMPER_FRONT: track 126.8 -> 109.0 mm
- net SW_OFF: track 39.9 -> 57.5 mm
- net JET_12V: track 60.3 -> 43.0 mm, vias 0 -> 1
- net TOF_FL_SCL: track 137.8 -> 120.6 mm, vias 0 -> 2
- net ENC2_A: track 137.8 -> 121.1 mm, vias 0 -> 2
- net ENC2_B: track 140.4 -> 155.7 mm, vias 0 -> 1
- net GPIO19: track 77.3 -> 90.8 mm
- net TOF_RL_SCL: track 188.1 -> 175.0 mm, vias 1 -> 0
- net GPIO13: track 96.4 -> 83.4 mm, vias 1 -> 3
- net I2C1_SDA: track 191.0 -> 201.9 mm, vias 3 -> 4
- net INA_IN4P: track 128.4 -> 118.8 mm, vias 2 -> 5
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Other:
- outline, holes or cut-outs redrawn

Commit message: wip(hw): body PCB rev B in progress (BLDC drive, on-board power, factory assembly)
Co-Authored-By: Claude Opus 5.5 <noreply@anthropic.com>
Claude-Session: https://claude.ai/code/session_01BqVLDBXG9mdqYKRp3kWsAJ
Parts:
- removed C1: 1000uF 35V, Capacitor_THT:CP_Radial_D12.5mm_P5.00mm
- removed C2: 100nF, Capacitor_SMD:C_0603_1608Metric
- removed F5: ATO 7.5A, rabbit_body:Fuseholder_ATO_Keystone_3557x2
- removed F6: ATO 2A, rabbit_body:Fuseholder_ATO_Keystone_3557x2
- removed F7: ATO (spare), rabbit_body:Fuseholder_ATO_Keystone_3557x2
- removed J19: USB hub 7-36V, Connector_JST:JST_XH_B2B-XH-A_1x02_P2.50mm_Vertical
- removed J2: RoboClaw B+/B-, rabbit_body:WirePads_2x_AWG14_P8.4mm
- removed J20: spare out, TerminalBlock_Phoenix:TerminalBlock_Phoenix_MKDS-1,5-2-5.08_1x02_P5.08mm_Horizontal
- removed J4: RoboClaw I/O, Connector_PinHeader_2.54mm:PinHeader_2x05_P2.54mm_Vertical
- removed J6: ENC left, Connector_JST:JST_XH_B4B-XH-A_1x04_P2.50mm_Vertical
- removed J7: ENC right, Connector_JST:JST_XH_B4B-XH-A_1x04_P2.50mm_Vertical
- removed R19, R21: 100k, Resistor_SMD:R_0603_1608Metric
- removed R20: 1k, Resistor_SMD:R_0603_1608Metric
- removed U2: Pololu 2813, rabbit_body:Pololu_BigPushbutton_HP
- removed U3: INA4235, rabbit_body:TI_DSBGA-16_YBJ_1.5x1.5mm_P0.4mm
- added C100: 1nF, Capacitor_SMD:C_0603_1608Metric, F.Cu at (123.0, 211.2)
- added C101: 1nF, Capacitor_SMD:C_0603_1608Metric, F.Cu at (124.6, 211.2)
- added C102: 1nF, Capacitor_SMD:C_0603_1608Metric, F.Cu at (126.2, 211.2)
- added C103: 1nF, Capacitor_SMD:C_0603_1608Metric, F.Cu at (159.0, 224.2)
- added C104: 1nF, Capacitor_SMD:C_0603_1608Metric, F.Cu at (160.6, 224.2)
- added C105: 1nF, Capacitor_SMD:C_0603_1608Metric, F.Cu at (162.2, 224.2)
- added C1101: 100nF, Capacitor_SMD:C_0603_1608Metric, F.Cu at (119.4, 260.4)
- added C1102: 100nF, Capacitor_SMD:C_0603_1608Metric, F.Cu at (117.8, 260.4)
- added C1103: 10uF 50V, Capacitor_SMD:C_1210_3225Metric, F.Cu at (115.6, 258.6)
- added C1104: 1uF, Capacitor_SMD:C_0402_1005Metric, F.Cu at (120.7, 257.3)
- added C1105: 47nF, Capacitor_SMD:C_0402_1005Metric, F.Cu at (119.7, 256.2)
- added C1106: 10uF, Capacitor_SMD:C_0805_2012Metric, F.Cu at (116.0, 253.6)
- added C1107: 1uF, Capacitor_SMD:C_0603_1608Metric, F.Cu at (128.6, 256.8)
- added C1109: 220uF 35V, Capacitor_SMD:CP_Elec_8x10.5, F.Cu at (104.5, 253.0)
- added C1110: 1nF, Capacitor_SMD:C_0603_1608Metric, F.Cu at (131.0, 223.5)
- added C1111: 1nF, Capacitor_SMD:C_0603_1608Metric, F.Cu at (131.0, 225.1)
- added C1112: 1nF, Capacitor_SMD:C_0603_1608Metric, F.Cu at (131.0, 226.7)
- added C120: 100nF, Capacitor_SMD:C_0603_1608Metric, F.Cu at (139.3, 227.8)
- added C1201: 100nF, Capacitor_SMD:C_0603_1608Metric, F.Cu at (171.4, 260.4)
- added C1202: 100nF, Capacitor_SMD:C_0603_1608Metric, F.Cu at (169.8, 260.4)
- added C1203: 10uF 50V, Capacitor_SMD:C_1210_3225Metric, F.Cu at (167.6, 258.6)
- added C1204: 1uF, Capacitor_SMD:C_0402_1005Metric, F.Cu at (172.7, 257.3)
- added C1205: 47nF, Capacitor_SMD:C_0402_1005Metric, F.Cu at (171.7, 256.2)
- added C1206: 10uF, Capacitor_SMD:C_0805_2012Metric, F.Cu at (168.0, 253.6)
- added C1207: 1uF, Capacitor_SMD:C_0603_1608Metric, F.Cu at (180.6, 256.8)
- added C1209: 220uF 35V, Capacitor_SMD:CP_Elec_8x10.5, F.Cu at (179.5, 243.0)
- added C121: 100nF, Capacitor_SMD:C_0603_1608Metric, F.Cu at (151.0, 231.7)
- added C1210: 1nF, Capacitor_SMD:C_0603_1608Metric, F.Cu at (131.0, 229.5)
- added C1211: 1nF, Capacitor_SMD:C_0603_1608Metric, F.Cu at (131.0, 231.1)
- added C1212: 1nF, Capacitor_SMD:C_0603_1608Metric, F.Cu at (131.0, 232.7)
- added C122: 100nF, Capacitor_SMD:C_0603_1608Metric, F.Cu at (154.7, 220.2)
- added C123: 100nF, Capacitor_SMD:C_0603_1608Metric, F.Cu at (143.2, 216.3)
- added C14A: 100nF, Capacitor_SMD:C_0603_1608Metric, F.Cu at (164.6, 226.0)
- added C14B: 100nF, Capacitor_SMD:C_0603_1608Metric, F.Cu at (170.6, 226.0)
- added C18: 2.2uF, Capacitor_SMD:C_0603_1608Metric, F.Cu at (167.8, 215.0)
- added C19: 100nF, Capacitor_SMD:C_0603_1608Metric, F.Cu at (169.8, 219.6)
- added C20: 100nF, Capacitor_SMD:C_0603_1608Metric, F.Cu at (195.4, 220.6)
- added C21: 100nF, Capacitor_SMD:C_0603_1608Metric, F.Cu at (195.4, 226.4)
- added C22: 100nF, Capacitor_SMD:C_0603_1608Metric, F.Cu at (188.4, 221.0)
- added C23: 47nF, Capacitor_SMD:C_0603_1608Metric, F.Cu at (195.3, 211.2)
- added C24: 10nF, Capacitor_SMD:C_0603_1608Metric, F.Cu at (188.4, 227.0)
- added C25: 1uF, Capacitor_SMD:C_0603_1608Metric, F.Cu at (192.3, 210.4)
- added C26: 100nF, Capacitor_SMD:C_0603_1608Metric, F.Cu at (184.8, 241.6)
- added C27: 100nF, Capacitor_SMD:C_0603_1608Metric, F.Cu at (189.0, 203.9)
- added C28: 100nF, Capacitor_SMD:C_0603_1608Metric, F.Cu at (184.4, 192.7)
- added C29: 100nF, Capacitor_SMD:C_0603_1608Metric, F.Cu at (173.2, 93.5)
- added C30: 220uF 35V, Capacitor_SMD:CP_Elec_8x10.5, F.Cu at (201.0, 187.5)
- added C31: 10uF 50V, Capacitor_SMD:C_1210_3225Metric, F.Cu at (195.5, 195.0)
- added C32: 10uF 50V, Capacitor_SMD:C_1210_3225Metric, F.Cu at (191.6, 195.0)
- added C33: 220uF 35V, Capacitor_SMD:CP_Elec_8x10.5, F.Cu at (187.5, 106.5)
- added C401: 10uF 50V, Capacitor_SMD:C_1210_3225Metric, F.Cu at (115.1, 103.3)
- added C402: 10uF 50V, Capacitor_SMD:C_1210_3225Metric, F.Cu at (124.9, 103.3)
- added C403: 470nF, Capacitor_SMD:C_0603_1608Metric, F.Cu at (117.5, 103.3)
- added C404: 470nF, Capacitor_SMD:C_0603_1608Metric, F.Cu at (122.5, 103.3)
- added C405: 100nF, Capacitor_SMD:C_0402_1005Metric, F.Cu at (117.5, 105.5)
- added C406: 1uF, Capacitor_SMD:C_0603_1608Metric, F.Cu at (118.7, 108.8)
- added C407: 100nF, Capacitor_SMD:C_0402_1005Metric, F.Cu at (117.0, 107.2)
- added C408: 10pF, Capacitor_SMD:C_0603_1608Metric, F.Cu at (120.0, 113.3)
- added C410: 22uF, Capacitor_SMD:C_1206_3216Metric, F.Cu at (114.0, 85.5)
- added C411: 22uF, Capacitor_SMD:C_1206_3216Metric, F.Cu at (117.0, 85.5)
- added C412: 22uF, Capacitor_SMD:C_1206_3216Metric, F.Cu at (120.0, 85.5)
- added C413: 22uF, Capacitor_SMD:C_1206_3216Metric, F.Cu at (123.0, 85.5)
- added C414: 22uF, Capacitor_SMD:C_1206_3216Metric, F.Cu at (126.0, 85.5)
- added C451: 1uF, Capacitor_SMD:C_0603_1608Metric, F.Cu at (129.7, 269.6)
- added C461: 1uF, Capacitor_SMD:C_0603_1608Metric, F.Cu at (170.3, 269.6)
- added C55: 1uF, Capacitor_SMD:C_0603_1608Metric, F.Cu at (134.4, 255.8)
- added C601: 10uF 50V, Capacitor_SMD:C_1210_3225Metric, F.Cu at (159.1, 103.3)
- added C602: 10uF 50V, Capacitor_SMD:C_1210_3225Metric, F.Cu at (168.9, 103.3)
- added C603: 470nF, Capacitor_SMD:C_0603_1608Metric, F.Cu at (161.4, 103.3)
- added C604: 470nF, Capacitor_SMD:C_0603_1608Metric, F.Cu at (166.6, 103.3)
- added C605: 100nF, Capacitor_SMD:C_0402_1005Metric, F.Cu at (161.6, 105.5)
- added C606: 1uF, Capacitor_SMD:C_0603_1608Metric, F.Cu at (162.7, 108.8)
- added C607: 100nF, Capacitor_SMD:C_0402_1005Metric, F.Cu at (161.0, 107.2)
- added C608: 10pF, Capacitor_SMD:C_0603_1608Metric, F.Cu at (164.0, 113.3)
- added C610: 22uF, Capacitor_SMD:C_1206_3216Metric, F.Cu at (158.0, 85.5)
- added C611: 22uF, Capacitor_SMD:C_1206_3216Metric, F.Cu at (161.0, 85.5)
- added C612: 22uF, Capacitor_SMD:C_1206_3216Metric, F.Cu at (164.0, 85.5)
- added C613: 22uF, Capacitor_SMD:C_1206_3216Metric, F.Cu at (167.0, 85.5)
- added C614: 22uF, Capacitor_SMD:C_1206_3216Metric, F.Cu at (170.0, 85.5)
- added C63: 100nF, Capacitor_SMD:C_0603_1608Metric, F.Cu at (145.4, 238.6)
- added C70: 100nF, Capacitor_SMD:C_0603_1608Metric, F.Cu at (194.6, 202.0)
- added C71: 100nF, Capacitor_SMD:C_0603_1608Metric, F.Cu at (176.2, 191.0)
- added C72: 100nF, Capacitor_SMD:C_0603_1608Metric, F.Cu at (154.7, 96.2)
- added C73: 100nF, Capacitor_SMD:C_0603_1608Metric, F.Cu at (177.7, 101.5)
- added C80: 47nF, Capacitor_SMD:C_0603_1608Metric, F.Cu at (134.8, 106.2)
- added C81: 100nF, Capacitor_SMD:C_0603_1608Metric, F.Cu at (138.5, 98.4)
- added C82: 1uF, Capacitor_SMD:C_0805_2012Metric, F.Cu at (146.6, 97.4)
- added C83: 100nF, Capacitor_SMD:C_0603_1608Metric, F.Cu at (155.0, 88.4)
- added C84: 4.7uF, Capacitor_SMD:C_0603_1608Metric, F.Cu at (137.6, 227.8)
- added C85: 1uF, Capacitor_SMD:C_0603_1608Metric, F.Cu at (147.8, 231.7)
- added C86: 10nF, Capacitor_SMD:C_0603_1608Metric, F.Cu at (147.8, 233.3)
- added C87: 100nF, Capacitor_SMD:C_0603_1608Metric, F.Cu at (137.6, 223.2)
- added C88: 18pF, Capacitor_SMD:C_0603_1608Metric, F.Cu at (133.6, 218.4)
- added C89: 18pF, Capacitor_SMD:C_0603_1608Metric, F.Cu at (133.6, 220.8)
- added C90: 1uF, Capacitor_SMD:C_0603_1608Metric, F.Cu at (160.2, 213.5)
- added C91: 4.7uF, Capacitor_SMD:C_0603_1608Metric, F.Cu at (153.8, 213.5)
- added D10: SMBJ20A, Diode_SMD:D_SMB, F.Cu at (134.0, 245.5)
- added D11: BZT52C12, Diode_SMD:D_SOD-123, F.Cu at (155.4, 257.0)
- added D12: BAT54S, Package_TO_SOT_SMD:SOT-23, F.Cu at (167.6, 226.0)
- added D13: SMBJ20A, Diode_SMD:D_SMB, F.Cu at (195.5, 119.5)
- added D14: SMBJ20A, Diode_SMD:D_SMB, F.Cu at (131.0, 81.0)
- added D8: BZT52C8V2, Diode_SMD:D_SOD-123, F.Cu at (186.0, 215.0)
- added D9: 1N4148WS, Diode_SMD:D_SOD-323, F.Cu at (188.9, 210.4)
- added D93: LED red, LED_SMD:LED_0603_1608Metric, F.Cu at (160.4, 209.4)
- added J41: motor phases, Connector_Molex:Molex_KK-396_A-41791-0003_1x03_P3.96mm_Vertical, F.Cu at (120.0, 279.5)
- added J42: motor phases, Connector_Molex:Molex_KK-396_A-41791-0003_1x03_P3.96mm_Vertical, F.Cu at (172.0, 279.5)
- added J43: Halls, Connector_JST:JST_PH_B5B-PH-K_1x05_P2.00mm_Vertical, F.Cu at (133.5, 279.5)
- added J44: Halls, Connector_JST:JST_PH_B5B-PH-K_1x05_P2.00mm_Vertical, F.Cu at (158.5, 279.5)
- added J45: encoder, Connector_JST:JST_GH_BM07B-GHS-TBT_1x07-1MP_P1.25mm_Vertical, F.Cu at (137.5, 270.3)
- added J46: encoder, Connector_JST:JST_GH_BM07B-GHS-TBT_1x07-1MP_P1.25mm_Vertical, F.Cu at (162.5, 270.3)
- added J47: SWD, Connector_PinHeader_1.27mm:PinHeader_2x05_P1.27mm_Vertical_SMD, F.Cu at (145.0, 210.6)
- added J48: RoboClaw S, Connector_JST:JST_XH_B4B-XH-A_1x04_P2.50mm_Vertical, F.Cu at (95.5, 190.0)
- added J49: MOT_BUS out, TerminalBlock_Phoenix:TerminalBlock_Phoenix_MKDS-1,5-2-5.08_1x02_P5.08mm_Horizontal, F.Cu at (97.0, 245.0)
- added JP1: UART0 TX, Jumper:SolderJumper-3_P1.3mm_Bridged12_RoundedPad1.0x1.5mm_NumberLabels, F.Cu at (114.0, 170.0)
- added JP2: UART0 RX, Jumper:SolderJumper-3_P1.3mm_Bridged12_RoundedPad1.0x1.5mm_NumberLabels, F.Cu at (114.0, 166.5)
- added JP3: S0 source, Jumper:SolderJumper-3_P1.3mm_Bridged12_RoundedPad1.0x1.5mm_NumberLabels, F.Cu at (140.0, 44.0)
- added L4: 3.3uH, Inductor_SMD:L_Coilcraft_XAL1010-XXX, F.Cu at (120.0, 95.0)
- added L6: 3.3uH, Inductor_SMD:L_Coilcraft_XAL1010-XXX, F.Cu at (164.0, 95.0)
- added Q4: MMBT3906, Package_TO_SOT_SMD:SOT-23, F.Cu at (188.0, 236.5)
- added Q5: AO3400A, Package_TO_SOT_SMD:SOT-23, F.Cu at (189.6, 215.0)
- added Q6: BSC026N04LS, Package_TO_SOT_SMD:TDSON-8-1, F.Cu at (150.0, 256.0)
- added Q7: AO3400A, Package_TO_SOT_SMD:SOT-23, F.Cu at (151.0, 101.6)
- added Q8: AO3400A, Package_TO_SOT_SMD:SOT-23, F.Cu at (148.5, 69.0)
- added R100: 1k, Resistor_SMD:R_0603_1608Metric, F.Cu at (123.0, 208.0)
- added R101: 1k, Resistor_SMD:R_0603_1608Metric, F.Cu at (124.6, 208.0)
- added R102: 1k, Resistor_SMD:R_0603_1608Metric, F.Cu at (126.2, 208.0)
- added R103: 1k, Resistor_SMD:R_0603_1608Metric, F.Cu at (159.0, 221.0)
- added R104: 1k, Resistor_SMD:R_0603_1608Metric, F.Cu at (160.6, 221.0)
- added R105: 1k, Resistor_SMD:R_0603_1608Metric, F.Cu at (162.2, 221.0)
- added R110: 4.7k, Resistor_SMD:R_0603_1608Metric, F.Cu at (123.0, 204.8)
- added R1101: 22, Resistor_SMD:R_0402_1005Metric, F.Cu at (120.7, 254.8)
- added R1102: 100, Resistor_SMD:R_0603_1608Metric, F.Cu at (128.0, 223.5)
- added R1103: 100, Resistor_SMD:R_0603_1608Metric, F.Cu at (128.0, 225.1)
- added R1104: 100, Resistor_SMD:R_0603_1608Metric, F.Cu at (128.0, 226.7)
- added R111: 4.7k, Resistor_SMD:R_0603_1608Metric, F.Cu at (124.6, 204.8)
- added R112: 4.7k, Resistor_SMD:R_0603_1608Metric, F.Cu at (126.2, 204.8)
- added R113: 4.7k, Resistor_SMD:R_0603_1608Metric, F.Cu at (159.0, 217.8)
- added R114: 4.7k, Resistor_SMD:R_0603_1608Metric, F.Cu at (160.6, 217.8)
- added R115: 4.7k, Resistor_SMD:R_0603_1608Metric, F.Cu at (162.2, 217.8)
- added R1201: 22, Resistor_SMD:R_0402_1005Metric, F.Cu at (172.7, 254.8)
- added R1202: 100, Resistor_SMD:R_0603_1608Metric, F.Cu at (128.0, 229.5)
- added R1203: 100, Resistor_SMD:R_0603_1608Metric, F.Cu at (128.0, 231.1)
- added R1204: 100, Resistor_SMD:R_0603_1608Metric, F.Cu at (128.0, 232.7)
- added R120A: 4.7k, Resistor_SMD:R_0603_1608Metric, F.Cu at (130.0, 27.0)
- added R120B: 4.7k, Resistor_SMD:R_0603_1608Metric, F.Cu at (133.2, 27.0)
- added R121A: 4.7k, Resistor_SMD:R_0603_1608Metric, F.Cu at (166.0, 27.0)
- added R121B: 4.7k, Resistor_SMD:R_0603_1608Metric, F.Cu at (169.2, 27.0)
- added R122A: 4.7k, Resistor_SMD:R_0603_1608Metric, F.Cu at (97.0, 258.5)
- added R122B: 4.7k, Resistor_SMD:R_0603_1608Metric, F.Cu at (100.2, 258.5)
- added R123A: 4.7k, Resistor_SMD:R_0603_1608Metric, F.Cu at (199.0, 270.5)
- added R123B: 4.7k, Resistor_SMD:R_0603_1608Metric, F.Cu at (202.2, 270.5)
- added R130: 22, Resistor_SMD:R_0603_1608Metric, F.Cu at (132.5, 237.0)
- added R131: 22, Resistor_SMD:R_0603_1608Metric, F.Cu at (134.1, 237.0)
- added R132: 22, Resistor_SMD:R_0603_1608Metric, F.Cu at (135.7, 237.0)
- added R133: 22, Resistor_SMD:R_0603_1608Metric, F.Cu at (157.5, 237.0)
- added R134: 22, Resistor_SMD:R_0603_1608Metric, F.Cu at (159.1, 237.0)
- added R135: 22, Resistor_SMD:R_0603_1608Metric, F.Cu at (160.7, 237.0)
- added R14B: 100k, Resistor_SMD:R_0603_1608Metric, F.Cu at (172.2, 226.0)
- added R32B: 1k, Resistor_SMD:R_0603_1608Metric, F.Cu at (150.0, 235.2)
- added R33B: 1k, Resistor_SMD:R_0603_1608Metric, F.Cu at (150.0, 236.8)
- added R401: 100k, Resistor_SMD:R_0603_1608Metric, F.Cu at (118.7, 111.7)
- added R402: 24k, Resistor_SMD:R_0603_1608Metric, F.Cu at (121.3, 111.7)
- added R403: 4.99k, Resistor_SMD:R_0603_1608Metric, F.Cu at (117.4, 113.3)
- added R404: 100k, Resistor_SMD:R_0603_1608Metric, F.Cu at (123.0, 108.5)
- added R405: 22k, Resistor_SMD:R_0603_1608Metric, F.Cu at (123.0, 110.1)
- added R406: 39k, Resistor_SMD:R_0603_1608Metric, F.Cu at (121.0, 109.2)
- added R40A: 330, Resistor_SMD:R_0603_1608Metric, F.Cu at (155.0, 75.5)
- added R41: 10k, Resistor_SMD:R_0603_1608Metric, F.Cu at (185.2, 224.0)
- added R42: 100, Resistor_SMD:R_0603_1608Metric, F.Cu at (196.9, 211.2)
- added R43: 100k, Resistor_SMD:R_0603_1608Metric, F.Cu at (184.8, 234.5)
- added R44: 22k, Resistor_SMD:R_0603_1608Metric, F.Cu at (184.8, 238.5)
- added R45: 47k, Resistor_SMD:R_0603_1608Metric, F.Cu at (188.0, 232.4)
- added R451: 10, Resistor_SMD:R_0805_2012Metric, F.Cu at (129.7, 265.8)
- added R46: 220k, Resistor_SMD:R_0603_1608Metric, F.Cu at (188.4, 228.6)
- added R461: 10, Resistor_SMD:R_0805_2012Metric, F.Cu at (170.3, 265.8)
- added R47: 47k, Resistor_SMD:R_0603_1608Metric, F.Cu at (186.0, 219.4)
- added R48: 1k, Resistor_SMD:R_0603_1608Metric, F.Cu at (185.6, 210.4)
- added R49: 1M, Resistor_SMD:R_0603_1608Metric, F.Cu at (192.3, 212.0)
- added R50: 39R 2W, Resistor_SMD:R_2512_6332Metric, F.Cu at (141.0, 247.5)
- added R51: 39R 2W, Resistor_SMD:R_2512_6332Metric, F.Cu at (147.0, 247.5)
- added R52: 39R 2W, Resistor_SMD:R_2512_6332Metric, F.Cu at (153.0, 247.5)
- added R53: 39R 2W, Resistor_SMD:R_2512_6332Metric, F.Cu at (159.0, 247.5)
- added R55: 100, Resistor_SMD:R_0603_1608Metric, F.Cu at (134.4, 254.2)
- added R56: 4.7k, Resistor_SMD:R_0603_1608Metric, F.Cu at (134.4, 262.6)
- added R57: 60.4k, Resistor_SMD:R_0603_1608Metric, F.Cu at (140.0, 261.0)
- added R58: 10k, Resistor_SMD:R_0603_1608Metric, F.Cu at (140.0, 262.6)
- added R59: 1.5M, Resistor_SMD:R_0603_1608Metric, F.Cu at (143.6, 261.0)
- added R60: 10k, Resistor_SMD:R_0603_1608Metric, F.Cu at (157.4, 257.0)
- added R601: 100k, Resistor_SMD:R_0603_1608Metric, F.Cu at (162.7, 111.7)
- added R602: 20k, Resistor_SMD:R_0603_1608Metric, F.Cu at (165.3, 111.7)
- added R603: 4.99k, Resistor_SMD:R_0603_1608Metric, F.Cu at (161.4, 113.3)
- added R604: 100k, Resistor_SMD:R_0603_1608Metric, F.Cu at (167.0, 108.5)
- added R605: 22k, Resistor_SMD:R_0603_1608Metric, F.Cu at (167.0, 110.1)
- added R606: 39k, Resistor_SMD:R_0603_1608Metric, F.Cu at (164.9, 109.2)
- added R61: 100k, Resistor_SMD:R_0603_1608Metric, F.Cu at (159.0, 257.0)
- added R62: 33k, Resistor_SMD:R_0603_1608Metric, F.Cu at (163.0, 239.0)
- added R63: 100k, Resistor_SMD:R_0603_1608Metric, F.Cu at (142.2, 238.6)
- added R64: 10k, Resistor_SMD:R_0603_1608Metric, F.Cu at (143.8, 238.6)
- added R65: 10k, Resistor_SMD:R_0603_1608Metric, F.Cu at (130.0, 238.6)
- added R66: 10k, Resistor_SMD:R_0603_1608Metric, F.Cu at (186.6, 248.5)
- added R701: 10, Resistor_SMD:R_0603_1608Metric, F.Cu at (191.4, 202.0)
- added R702: 10, Resistor_SMD:R_0603_1608Metric, F.Cu at (193.0, 202.0)
- added R711: 10, Resistor_SMD:R_0603_1608Metric, F.Cu at (173.0, 191.0)
- added R712: 10, Resistor_SMD:R_0603_1608Metric, F.Cu at (174.6, 191.0)
- added R721: 10, Resistor_SMD:R_0603_1608Metric, F.Cu at (151.5, 96.2)
- added R722: 10, Resistor_SMD:R_0603_1608Metric, F.Cu at (153.1, 96.2)
- added R731: 10, Resistor_SMD:R_0603_1608Metric, F.Cu at (174.5, 101.5)
- added R732: 10, Resistor_SMD:R_0603_1608Metric, F.Cu at (176.1, 101.5)
- added R80: 68k, Resistor_SMD:R_0603_1608Metric, F.Cu at (138.0, 104.6)
- added R81: 10k, Resistor_SMD:R_0603_1608Metric, F.Cu at (136.4, 104.6)
- added R82: 150k, Resistor_SMD:R_0603_1608Metric, F.Cu at (138.0, 107.8)
- added R83: 10k, Resistor_SMD:R_0603_1608Metric, F.Cu at (136.4, 107.8)
- added R84: 3.9k, Resistor_SMD:R_0603_1608Metric, F.Cu at (150.0, 106.0)
- added R86: 1k, Resistor_SMD:R_0603_1608Metric, F.Cu at (154.4, 101.6)
- added R87: 100k, Resistor_SMD:R_0603_1608Metric, F.Cu at (151.0, 98.6)
- added R89: 220, Resistor_SMD:R_0603_1608Metric, F.Cu at (137.4, 44.0)
- added R90: 10k, Resistor_SMD:R_0603_1608Metric, F.Cu at (137.5, 215.0)
- added R91: 1k, Resistor_SMD:R_0603_1608Metric, F.Cu at (137.5, 213.4)
- added R92: 1k, Resistor_SMD:R_0603_1608Metric, F.Cu at (137.5, 211.8)
- added R93: 1k, Resistor_SMD:R_0603_1608Metric, F.Cu at (157.0, 209.4)
- added R94: 5.1k, Resistor_SMD:R_0603_1608Metric, F.Cu at (157.0, 233.0)
- added R95: 10k, Resistor_SMD:R_0603_1608Metric, F.Cu at (158.6, 233.0)
- added R96: 100k, Resistor_SMD:R_0603_1608Metric, F.Cu at (160.2, 233.0)
- added R97: 100k, Resistor_SMD:R_0603_1608Metric, F.Cu at (161.8, 233.0)
- added R98: 100k, Resistor_SMD:R_0603_1608Metric, F.Cu at (163.4, 233.0)
- added R99: 10k, Resistor_SMD:R_0603_1608Metric, F.Cu at (165.0, 233.0)
- added R9A: 10k, Resistor_SMD:R_0603_1608Metric, F.Cu at (166.6, 233.0)
- added RT65: NTC 10k, Resistor_SMD:R_0603_1608Metric, F.Cu at (130.0, 251.5)
- added RT66: NTC 10k, Resistor_SMD:R_0603_1608Metric, F.Cu at (184.0, 251.5)
- added TP10: +3V3_MCU, TestPoint:TestPoint_THTPad_D1.5mm_Drill0.7mm, F.Cu at (131.0, 211.0)
- added TP11: GND_MOT, TestPoint:TestPoint_THTPad_D1.5mm_Drill0.7mm, F.Cu at (110.0, 262.0)
- added TP12: BAT_F, TestPoint:TestPoint_THTPad_D1.5mm_Drill0.7mm, F.Cu at (187.0, 242.0)
- added TP9: MOT_BUS, TestPoint:TestPoint_THTPad_D1.5mm_Drill0.7mm, F.Cu at (113.5, 241.0)
- added U10: LM74800, rabbit_body:TI_DRR0012E_WSON-12_3x3mm_P0.5mm_EP1.3x2.5mm, F.Cu at (192.0, 223.5)
- added U11: DRV8316CR, rabbit_body:TI_RGF0040E_VQFN-40_5x7mm_P0.5mm_EP3.7x5.7mm, F.Cu at (124.0, 256.0)
- added U12: DRV8316CR, rabbit_body:TI_RGF0040E_VQFN-40_5x7mm_P0.5mm_EP3.7x5.7mm, F.Cu at (176.0, 256.0)
- added U15: TLV75533, Package_TO_SOT_SMD:SOT-23-5, F.Cu at (157.0, 213.5)
- added U16: SN74LVC1G132, Package_TO_SOT_SMD:SOT-23-5, F.Cu at (166.6, 219.6)
- added U17: LM393, Package_SO:SOIC-8_3.9x4.9mm_P1.27mm, F.Cu at (140.0, 256.5)
- added U18: TL431, Package_TO_SOT_SMD:SOT-23, F.Cu at (134.4, 259.6)
- added U19: INA226, Package_SO:MSOP-10_3x3mm_P0.5mm, F.Cu at (154.0, 92.0)
- added U20: INA226, Package_SO:MSOP-10_3x3mm_P0.5mm, F.Cu at (177.5, 93.5)
- added U21: INA226, Package_SO:MSOP-10_3x3mm_P0.5mm, F.Cu at (192.0, 206.4)
- added U22: INA226, Package_SO:MSOP-10_3x3mm_P0.5mm, F.Cu at (182.0, 190.0)
- added Y1: 8MHz, Crystal:Crystal_SMD_3225-4Pin_3.2x2.5mm, F.Cu at (137.4, 219.6)
- BT1: footprint Battery:BatteryHolder_Keystone_3001_1x12mm -> Battery:BatteryHolder_Keystone_3000_1x12mm
- D2, D3, D4, D5, D6: value LED green -> LED red
- F1: value ATO 15A -> 15A; footprint rabbit_body:Fuseholder_ATO_Keystone_3557x2 -> rabbit_body:Fuse_Littelfuse_NANO2_451_2410
- F2: value ATO 10A -> 8A; footprint rabbit_body:Fuseholder_ATO_Keystone_3557x2 -> rabbit_body:Fuse_Littelfuse_NANO2_451_2410
- F3, F4: value ATO 5A -> 5A; footprint rabbit_body:Fuseholder_ATO_Keystone_3557x2 -> rabbit_body:Fuse_Littelfuse_NANO2_451_2410
- Q1, Q2: value AO3400A -> BSC010N04LS; footprint Package_TO_SOT_SMD:SOT-23 -> Package_TO_SOT_SMD:TDSON-8-1
- R17: value 100k -> 10k
- R18: value 1k -> 100k
- R2, R4: value 10mR 2W -> 10mR 1W
- R40: value 330 -> 150k
- TP4: value JET_12V -> JET_PWR
- U1: value RoboClaw 2x30A -> STM32G474RET6; footprint rabbit_body:RoboClaw_2x30A -> Package_QFP:LQFP-64_10x10mm_P0.5mm
- U4: value D24V90F5 -> LM61495; footprint rabbit_body:Pololu_D24V90F5 -> rabbit_body:TI_RPH0016B_VQFN-HR-16_3.5x4.5mm
- U5: value D36V50F12 -> TPS16630; footprint rabbit_body:Pololu_D36V50Fx -> Package_SO:HTSSOP-20-1EP_4.4x6.5mm_P0.65mm_EP3.4x6.5mm_Mask2.96x2.96mm_ThermalVias
- U6: value D36V50F6 -> LM61495; footprint rabbit_body:Pololu_D36V50Fx -> rabbit_body:TI_RPH0016B_VQFN-HR-16_3.5x4.5mm
- moved Q2 152.5 mm to (200.0, 216.5), turned to -90 degrees
- moved R40 148.0 mm to (186.8, 224.0)
- moved F3 145.2 mm to (109.4, 113.0), turned to 0 degrees
- moved Q1 133.7 mm to (200.0, 230.0), turned to 90 degrees
- moved F4 121.6 mm to (178.0, 111.5)
- moved R17 72.3 mm to (164.6, 215.0)
- moved R3 57.5 mm to (177.0, 198.5)
- moved F2 55.8 mm to (186.0, 198.5)
- moved TP2 51.9 mm to (130.1, 105.0)
- moved U4 51.0 mm to (120.0, 105.0)
- moved D5 35.1 mm to (206.6, 211.0), turned to 90 degrees
- moved D2 34.1 mm to (103.0, 116.0), turned to -90 degrees
- moved R36 34.1 mm to (103.0, 119.5)
- moved R4 32.1 mm to (145.0, 93.0), turned to 0 degrees
- moved TP4 32.1 mm to (140.0, 86.2)
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Connections:
- net JET_12V renamed JET_PWR
- net MOT_FUSED renamed MOT_F
- D1 pad 1: SW_OUT -> VBUS
- D7 pad 1: BAT_FUSED -> BAT_F
- F1 pad 2: BAT_FUSED -> BAT_F
- F4 pad 2: BRAIN_IN -> STEER_IN
- J3 pad 27: (no net) -> GPIO0
- J3 pad 28: (no net) -> GPIO1
- J5 pad 2: ESTOP_RC -> ESTOP
- Q1 pad 1: Q1_G -> BAT_F
- Q1 pad 2: GND -> BAT_F
- Q1 pad 3: JET_EN -> BAT_F
- Q2 pad 1: Q2_G -> VBUS_RAW
- Q2 pad 2: GND -> VBUS_RAW
- Q2 pad 3: TOF_EN -> VBUS_RAW
- R1 pad 1: SW_OUT -> VBUS_RAW
- R1 pad 3: INA_IN1P -> SH1_P
- R1 pad 4: INA_IN1N -> SH1_N
- R10 pad 2: RC_S1 -> UART0_TX
- R11 pad 1: RC_S2 -> UART0_RX
- R17 pad 1: GPIO16 -> ESTOP
- R18 pad 1: GPIO17 -> ESTOP
- R18 pad 2: SW_OFF -> ESTOP_DLY
- R2 pad 3: INA_IN2P -> SH2_P
- R2 pad 4: INA_IN2N -> SH2_N
- R22 pad 2: Q2_G -> Q8_G
- R23 pad 1: Q2_G -> Q8_G
- R3 pad 2: MOT_BAT -> MOT_BUS
- R3 pad 3: INA_IN3P -> SH3_P
- R3 pad 4: INA_IN3N -> SH3_N
- R32 pad 2: PWM0 -> PWM0_PCA
- R39 pad 1: VBUS -> LEDB_A
- R39 pad 2: LEDB_A -> VBUS
- R4 pad 1: 12V_RAW -> JET_OUT
- R4 pad 3: INA_IN4P -> SH4_P
- R4 pad 4: INA_IN4N -> SH4_N
- R40 pad 1: +3V3_TOF -> LM_SW
- R40 pad 2: LED33_A -> LM_OV
Routing:
- net +3V3_MCU: track 0.00 -> 265.2 mm, vias 0 -> 8
- net STEER_IN: track 213.9 -> 1.90 mm, vias 0 -> 5
- net SERVO_MCU: track 0.00 -> 205.1 mm, vias 0 -> 4
- net BRAIN_IN: track 197.2 -> 0.00 mm
- net BUMPER_FRONT: track 109.0 -> 267.2 mm, vias 1 -> 2
- net ENC2_B: track 155.7 -> 0.00 mm, vias 1 -> 0
- net GND: track 68.0 -> 219.0 mm, vias 50 -> 177
- net BODY_IN: track 146.4 -> 1.90 mm, vias 0 -> 5
- net RC_5V: track 144.4 -> 0.00 mm, vias 1 -> 0
- net INA_IN4N: track 130.3 -> 0.00 mm, vias 4 -> 0
- net +5V: track 317.8 -> 439.2 mm, vias 0 -> 15
- net ENC2_A: track 121.1 -> 0.00 mm, vias 2 -> 0
- net INA_IN4P: track 118.8 -> 0.00 mm, vias 5 -> 0
- net INA_ALERT: track 77.6 -> 195.9 mm
- net DRV_NSLEEP: track 0.00 -> 117.7 mm, vias 0 -> 4
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- added copper zone on F.Cu, net +5V
- added copper zone on F.Cu, net 6V_RAW
- added copper zone on B.Cu, net BAT_F
- added copper zone on F.Cu, net BAT_F
- added copper zone on B.Cu, net BODY_IN
- added copper zone on F.Cu, net BODY_IN
- added copper zone on F.Cu, net BRK_D
- added copper zone on F.Cu, net GND_MOT
- added copper zone on In1.Cu, net GND_MOT
- added copper zone on F.Cu, net JET_OUT
- added copper zone on B.Cu, net JET_PWR
- added copper zone on F.Cu, net JET_PWR
- added copper zone on B.Cu, net MOT_BUS
- added copper zone on F.Cu, net MOT_BUS
- added copper zone on B.Cu, net STEER_IN
- added copper zone on F.Cu, net STEER_IN
- added copper zone on F.Cu, net SW4
- added copper zone on F.Cu, net SW6
- added copper zone on B.Cu, net SW_MID
- added copper zone on F.Cu, net SW_MID
- added copper zone on B.Cu, net VBUS_RAW
- added copper zone on F.Cu, net VBUS_RAW
- removed copper zone on B.Cu, net BAT_FUSED
- removed copper zone on F.Cu, net BAT_FUSED
- removed copper zone on F.Cu, net MOT_BAT
- removed copper zone on B.Cu, net SW_OUT
- removed copper zone on F.Cu, net SW_OUT
Other:
- board text added: "3V3M"
- board text added: "BAT"
- board text added: "F1 15A"
- board text added: "F2 MOTORS 8A"
- board text added: "F3 5V 5A"
- board text added: "F4 6V 5A"
- board text added: "GNDM"
- board text added: "J21 JETSON 9-20V"
- board text added: "J41 MOTOR L"
- board text added: "J42 MOTOR R"
- board text added: "J43 HALL L"
- board text added: "J44 HALL R"
- board text added: "J45 ENC L A/B/Z or SSI"
- board text added: "J46 ENC R A/B/Z or SSI"
- board text added: "J47 SWD"
- board text added: "J48 ROBOCLAW S"
- board text added: "J49 VMOT OUT"
- board text added: "JET"
- board text added: "RABBIT 2.0 BODY rev B 2026-10"
- board text added: "U1 MOTOR MCU"
- board text added: "U10 POWER SWITCH"
- board text added: "U11 DRV8316 L"
- board text added: "U12 DRV8316 R"
- board text added: "U19 INA JET 0x46"
- board text added: "U20 INA 6V 0x44"
- board text added: "U21 INA BAT 0x41"
- board text added: "U22 INA MOT 0x45"
- board text added: "U4 5.2V BUCK"
- board text added: "U5 JETSON EFUSE"
- board text added: "U6 6V SERVO BUCK"
- board text added: "VMOT"
- board text added: "rev B"
- board text removed: "12V"
- board text removed: "F1 MAIN 15A"
- board text removed: "F2 MOTORS 10A"
- board text removed: "F3 BODY 5V 5A"
- board text removed: "F4 JETSON 5A"
- board text removed: "F5 SERVO 7.5A"
- board text removed: "F6 USB HUB 2A"
- board text removed: "F7 SPARE"
- board text removed: "J19 USB HUB PWR"
- board text removed: "J20 SPARE BAT OUT"
- board text removed: "J21 JETSON 12V"
- board text removed: "J4 ROBOCLAW I/O"
- board text removed: "J6 ENC L (M1)"
- board text removed: "J7 ENC R (M2)"
- board text removed: "RABBIT 2.0 BODY rev A 2026-10"
