File: pcb/rabbit-body/rabbit-body.kicad_pcb (KiCad board)
At the start: 4 copper layers, 120.5 x 269.9 mm, 346 parts, among them J1 XT60 BAT, J10 ToF, J11 ToF, J12 lidar C1, J13 bumpers front, J14 bumpers rear, J15 button, J16 status LED, J17 Jetson UART, J18 Pi fan 5V, J21 XT30 JETSON, J22 servo 0, J23 servo 1, J24 servo 2, J25 servo 3, J3 Pi 40-pin, J41 motor phases, J42 motor phases, J43 Halls, J44 Halls, J45 encoder, J46 encoder, J47 SWD, J48 RoboClaw S, J49 MOT_BUS out, J5 E-stop loop, J8 ToF, J9 ToF, Q1 BSC010N04LS, Q2 BSC010N04LS, Q3 AO3400A, Q4 MMBT3906, Q5 AO3400A, Q6 BSC026N04LS, Q7 AO3400A, Q8 AO3400A, U1 STM32G474RET6, U10 LM74800, U11 DRV8316CR, U12 DRV8316CR, U15 TLV75533, U16 SN74LVC1G132, U17 LM393, U18 TL431, U19 INA226, U20 INA226, U21 INA226, U22 INA226, U4 LM61495, U5 TPS16630, U6 LM61495, U7 TPS73733, U8 PCA9685PW, U9 DS3231SN, Y1 8MHz

Commit message: wip(hw): body PCB rev B, state when paused
Co-Authored-By: Claude Opus 5.5 <noreply@anthropic.com>
Claude-Session: https://claude.ai/code/session_01BqVLDBXG9mdqYKRp3kWsAJ
Parts:
- moved R451 64.6 mm to (164.0, 211.0)
- moved R461 55.0 mm to (166.0, 211.0)
Routing:
- net +3V3_TOF: track 494.7 -> 0.00 mm, vias 1 -> 0
- net +3V3_PI: track 468.3 -> 14.8 mm, vias 13 -> 2
- net BUMPER_FRONT: track 267.2 -> 0.00 mm, vias 2 -> 0
- net +3V3_MCU: track 265.2 -> 0.00 mm, vias 8 -> 0
- net I2C1_SCL: track 259.8 -> 0.00 mm, vias 8 -> 0
- net I2C1_SDA: track 258.8 -> 0.00 mm, vias 7 -> 0
- net BTN_ON: track 212.3 -> 0.00 mm, vias 1 -> 0
- net SERVO_MCU: track 205.1 -> 0.00 mm, vias 4 -> 0
- net INA_ALERT: track 195.9 -> 0.00 mm, vias 1 -> 0
- net BUMPER_REAR: track 193.0 -> 0.00 mm, vias 1 -> 0
- net TOF_RR_SCL: track 190.3 -> 0.00 mm
- net TOF_RR_SDA: track 189.5 -> 0.00 mm, vias 1 -> 0
- net TOF_RL_SCL: track 182.2 -> 0.00 mm, vias 2 -> 0
- net TOF_RL_SDA: track 171.9 -> 0.00 mm, vias 1 -> 0
- net TOF_FL_SDA: track 132.5 -> 0.00 mm, vias 1 -> 0
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