File: pcb/rabbit-body/rabbit-body.kicad_pcb (KiCad board)
At the start: 4 copper layers, 120.5 x 269.9 mm, 346 parts, among them J1 XT60 BAT, J10 ToF, J11 ToF, J12 lidar C1, J13 bumpers front, J14 bumpers rear, J15 button, J16 status LED, J17 Jetson UART, J18 Pi fan 5V, J21 XT30 JETSON, J22 servo 0, J23 servo 1, J24 servo 2, J25 servo 3, J3 Pi 40-pin, J41 motor phases, J42 motor phases, J43 Halls, J44 Halls, J45 encoder, J46 encoder, J47 SWD, J48 RoboClaw S, J49 MOT_BUS out, J5 E-stop loop, J8 ToF, J9 ToF, Q1 BSC010N04LS, Q2 BSC010N04LS, Q3 AO3400A, Q4 MMBT3906, Q5 AO3400A, Q6 BSC026N04LS, Q7 AO3400A, Q8 AO3400A, U1 STM32G474RET6, U10 LM74800, U11 DRV8316CR, U12 DRV8316CR, U15 TLV75533, U16 SN74LVC1G132, U17 LM393, U18 TL431, U19 INA226, U20 INA226, U21 INA226, U22 INA226, U4 LM61495, U5 TPS16630, U6 LM61495, U7 TPS73733, U8 PCA9685PW, U9 DS3231SN, Y1 8MHz

Commit message: feat(hw): body board rev C (8 layers, routed), ToF carrier, BLDC drop-in, datasheets
Co-Authored-By: Claude Opus 5.5 <noreply@anthropic.com>
Routing:
- net +3V3_TOF: track 0.00 -> 498.0 mm
- net +3V3_PI: track 14.8 -> 483.6 mm, vias 2 -> 10
- net +3V3_MCU: track 0.00 -> 285.3 mm, vias 0 -> 6
- net BUMPER_FRONT: track 0.00 -> 265.2 mm, vias 0 -> 2
- net I2C1_SCL: track 0.00 -> 252.9 mm, vias 0 -> 5
- net I2C1_SDA: track 0.00 -> 251.5 mm, vias 0 -> 6
- net SERVO_MCU: track 0.00 -> 220.2 mm, vias 0 -> 4
- net BUMPER_REAR: track 0.00 -> 192.1 mm, vias 0 -> 2
- net BTN_ON: track 0.00 -> 188.9 mm, vias 0 -> 2
- net TOF_RL_SDA: track 0.00 -> 185.2 mm, vias 0 -> 1
- net TOF_RR_SCL: track 0.00 -> 182.8 mm, vias 0 -> 1
- net TOF_RR_SDA: track 0.00 -> 179.7 mm
- net INA_ALERT: track 0.00 -> 176.8 mm, vias 0 -> 4
- net TOF_RL_SCL: track 0.00 -> 176.3 mm, vias 0 -> 2
- net TOF_FL_SCL: track 0.00 -> 164.9 mm, vias 0 -> 1
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